Commit message: rename all, and fix tf

File: urdf/ros2_control.xacro (robot description, xacro)
@@ -17,5 +17,5 @@
   <gazebo>
     <plugin filename="libgazebo_ros2_control.so" name="gazebo_ros2_control">
-      <parameters>$(find tricycle_test)/config/tricycle_drive_controller.yaml</parameters>
+      <parameters>$(find warehouse_bot)/config/tricycle_drive_controller.yaml</parameters>
     </plugin>
   </gazebo>

File: urdf/warehouse_bot.xacro (robot description, xacro)
@@ -1,5 +1,5 @@
 <?xml version="1.0"?>
 <robot name="tricycle_drive" xmlns:xacro="http://ros.org/wiki/xacro">
-  <xacro:include filename="$(find tricycle_test)/urdf/ros2_control.xacro" />
+  <xacro:include filename="$(find warehouse_bot)/urdf/ros2_control.xacro" />
   <material name="Black">
     <color rgba="0 0 0 1" />
@@ -18,24 +18,24 @@
   <link name="chassis">
     <visual>
-      <origin xyz="-0.8 0 -0.2" rpy="0 0 0"/>
+      <origin xyz="0 0 -0.04" rpy="0 0 0"/>
       <geometry>
-        <mesh filename="file://$(find tricycle_test)/meshes/chassis.stl" scale="0.002 0.002 0.002"/>
+        <mesh filename="file://$(find warehouse_bot)/meshes/chassis.stl" scale="0.002 0.002 0.002"/>
       </geometry>
       <material name="silver"/>
     </visual>
     <collision>
-      <origin xyz="-0.8 0 -0.2" rpy="0 0 0"/>
+      <origin xyz="0 0 -0.04" rpy="0 0 0"/>
       <geometry>
-        <mesh filename="file://$(find tricycle_test)/meshes/chassis.stl" scale="0.002 0.002 0.002"/>
+        <mesh filename="file://$(find warehouse_bot)/meshes/chassis.stl" scale="0.002 0.002 0.002"/>
       </geometry>
     </collision>
     <inertial>
       <origin xyz="0 0 0" rpy="0 0 0" />
-      <mass value="1" />
+      <mass value="70" />
       <inertia ixx="0.126164" ixy="0.0" ixz="0.0" iyy="0.416519" iyz="0.0" izz="0.481014" />
     </inertial>
   </link>
   <joint name="chassis_joint" type="fixed">
-    <origin xyz="0 0 0.5" rpy="0 0 0" />
+    <origin xyz="0 0 0" rpy="0 0 0" />
     <parent link="base_link" />
     <child link="chassis" />
@@ -45,20 +45,20 @@
     <collision>
       <geometry>
-        <cylinder length="0.08" radius="0.1" />
+        <cylinder length="0.08" radius="0.15" />
       </geometry>
     </collision>
     <visual>
       <geometry>
-        <cylinder length="0.08" radius="0.1" />
+        <cylinder length="0.08" radius="0.15" />
       </geometry>
       <material name="Black" />
     </visual>
     <inertial>
-      <mass value="2" />
+      <mass value="10" />
       <inertia ixx="0.145833" ixy="0.0" ixz="0.0" iyy="0.145833" iyz="0.0" izz="0.125" />
     </inertial>
   </link>
   <joint name="left_wheel_joint" type="continuous">
-    <origin xyz="-0.8 0.4 -0.2" rpy="-1.57 0 0" />
+    <origin xyz="0 0.4 0" rpy="-1.57 0 0" />
     <parent link="chassis" />
     <child link="left_wheel" />
@@ -70,20 +70,20 @@
     <collision>
       <geometry>
-        <cylinder length="0.08" radius="0.1" />
+        <cylinder length="0.08" radius="0.15" />
       </geometry>
     </collision>
     <visual>
       <geometry>
-        <cylinder length="0.08" radius="0.1" />
+        <cylinder length="0.08" radius="0.15" />
       </geometry>
       <material name="Black" />
     </visual>
     <inertial>
-      <mass value="2" />
+      <mass value="10" />
       <inertia ixx="0.145833" ixy="0.0" ixz="0.0" iyy="0.145833" iyz="0.0" izz="0.125" />
     </inertial>
   </link>
   <joint name="right_wheel_joint" type="continuous">
-    <origin xyz="-0.8 -0.4 -0.2" rpy="-1.57 0 0" />
+    <origin xyz="0 -0.4 0" rpy="-1.57 0 0" />
     <parent link="chassis" />
     <child link="right_wheel" />
@@ -106,5 +106,5 @@
   </link>
   <joint name="steering_joint" type="continuous">
-    <origin xyz="0.9 0 -0.2" rpy="0 0 0" />
+    <origin xyz="2.2 0 0" rpy="0 0 0" />
     <parent link="chassis" />
     <child link="steering_link" />
@@ -115,5 +115,5 @@
     <visual>
       <geometry>
-        <cylinder length="0.08" radius="0.1" />
+        <cylinder length="0.08" radius="0.15" />
       </geometry>
       <material name="Black" />
@@ -121,10 +121,10 @@
     <inertial>
       <origin xyz="0 0 0" rpy="0 0 0" />
-      <mass value="15" />
+      <mass value="20" />
       <inertia ixx="1" ixy="0" ixz="0" iyy="1" iyz="0" izz="1" />
     </inertial>
     <collision>
       <geometry>
-        <cylinder length="0.08" radius="0.1" />
+        <cylinder length="0.08" radius="0.15" />
       </geometry>
     </collision>
