Commit message: add

File: urdf/robot.urdf.xacro (robot description, xacro)
@@ -2,5 +2,5 @@
 <robot xmlns:xacro="http://www.ros.org/wiki/xacro"  name="robot">
     <xacro:include filename="warehouse_bot.xacro" />
-    <xacro:include filename="gazebo_control.xacro" />
     <xacro:include filename="ros2_control.xacro" />
+    <xacro:include filename="lidar.xacro" />
 </robot>

File: urdf/warehouse_bot.xacro (robot description, xacro)
@@ -40,5 +40,5 @@
         <origin xyz="0 0 0" rpy="0 0 0" />
         <mass value="70" />
-        <inertia ixx="2.5" ixy="0.0" ixz="0.0" iyy="1.5" iyz="0.0" izz="3.7" />
+        <inertia ixx="0.126164" ixy="0.0" ixz="0.0" iyy="0.416519" iyz="0.0" izz="0.481014" />
       </inertial>
     </link>
@@ -62,5 +62,5 @@
       </visual>
       <inertial>
-        <mass value="10" />
+        <mass value="50" />
         <inertia ixx="0.145833" ixy="0.0" ixz="0.0" iyy="0.145833" iyz="0.0" izz="0.125" />
       </inertial>
@@ -87,5 +87,5 @@
       </visual>
       <inertial>
-        <mass value="10" />
+        <mass value="50" />
         <inertia ixx="0.145833" ixy="0.0" ixz="0.0" iyy="0.145833" iyz="0.0" izz="0.125" />
       </inertial>
@@ -108,6 +108,6 @@
       <inertial>
         <origin xyz="0 0 0" rpy="0 0 0" />
-        <mass value="40" />
-        <inertia ixx="0.01" ixy="0.0" ixz="0.0" iyy="0.01" iyz="0.0" izz="0.01" />
+        <mass value="1" />
+        <inertia ixx="0.1" ixy="0.0" ixz="0.0" iyy="0.1" iyz="0.0" izz="0.1" />
       </inertial>
     </link>
@@ -122,5 +122,5 @@
       <visual>
         <geometry>
-          <cylinder length="0.04" radius="0.075" />
+          <cylinder length="0.05" radius="0.075" />
         </geometry>
         <material name="Black" />
@@ -128,10 +128,10 @@
       <inertial>
         <origin xyz="0 0 0" rpy="0 0 0" />
-        <mass value="20" />
-        <inertia ixx="0.01" ixy="0" ixz="0" iyy="0.01" iyz="0" izz="0.01" />
+        <mass value="100" />
+        <inertia ixx="1" ixy="0" ixz="0" iyy="1" iyz="0" izz="1" />
       </inertial>
       <collision>
         <geometry>
-          <cylinder length="0.04" radius="0.075" />
+          <cylinder length="0.05" radius="0.075" />
         </geometry>
       </collision>
@@ -147,5 +147,5 @@
       <origin xyz="0 0 0" rpy="0 0 0"/>
       <mass value="0.01"/>
-      <inertia ixx="0.000238" iyy="3.5e-05" izz="0.00024" ixy="-0.0" iyz="-0.0" ixz="-0.0"/>
+        <inertia ixx="1.0" ixy="0.0" ixz="0.0" iyy="1.0" iyz="0.0" izz="1.0" />
     </inertial>
     <visual>
@@ -167,5 +167,5 @@
       <origin xyz="0 0 0" rpy="0 0 0"/>
       <mass value="0.01"/>
-      <inertia ixx="0.000238" iyy="3.5e-05" izz="0.00024" ixy="-0.0" iyz="-0.0" ixz="-0.0"/>
+        <inertia ixx="1.0" ixy="0.0" ixz="0.0" iyy="1.0" iyz="0.0" izz="1.0" />
     </inertial>
     <visual>
@@ -187,8 +187,8 @@
       <origin xyz="0 0 0" rpy="0 0 0"/>
       <mass value="0.01"/>
-      <inertia ixx="0.000238" iyy="3.5e-05" izz="0.00024" ixy="-0.0" iyz="-0.0" ixz="-0.0"/>
-    </inertial>
-    <visual>
-      <origin xyz="-1.0 0 -1.77" rpy="0 0 0"/>
+        <inertia ixx="1.0" ixy="0.0" ixz="0.0" iyy="1.0" iyz="0.0" izz="1.0" />
+    </inertial>
+    <visual>
+      <origin xyz="-1.0 0.0 -1.77" rpy="0 0 0"/>
       <geometry>
         <mesh filename="file://$(find warehouse_bot)/meshes/Intel_Realsense_D435_3.stl" scale="0.001 0.001 0.001"/>
@@ -197,5 +197,5 @@
     </visual>
     <collision>
-      <origin xyz="-1.0 0 -1.77" rpy="0 0 0"/>
+      <origin xyz="-1.0 0.0 -1.77" rpy="0 0 0"/>
       <geometry>
         <mesh filename="file://$(find warehouse_bot)/meshes/Intel_Realsense_D435_3.stl" scale="0.001 0.001 0.001"/>
@@ -203,5 +203,5 @@
     </collision>
   </link>
-  <link name="line_lidar_1">
+  <!-- <link name="line_lidar_1">
     <inertial>
       <origin xyz="0 0 0" rpy="0 0 0"/>
@@ -210,5 +210,5 @@
     </inertial>
     <visual>
-      <origin xyz="-1.1 0 2.29" rpy="3.14 0 0"/>
+      <origin xyz="-1.1 0.0 -2.3" rpy="0 0 0"/>
       <geometry>
         <mesh filename="file://$(find warehouse_bot)/meshes/16line_lidar_1.stl" scale="0.001 0.001 0.001"/>
@@ -217,18 +217,18 @@
     </visual>
     <collision>
-      <origin xyz="-1.1 0 2.29" rpy="3.14 0 0"/>
+      <origin xyz="-1.1 0.0 -2.3" rpy="0 0 0"/>
       <geometry>
         <mesh filename="file://$(find warehouse_bot)/meshes/16line_lidar_1.stl" scale="0.001 0.001 0.001"/>
       </geometry>
     </collision>
-  </link>
+  </link> -->
   <link name="mid-360-asm_1">
     <inertial>
       <origin xyz="0 0 0" rpy="0 0 0"/>
       <mass value="0.01"/>
-      <inertia ixx="0.00052" iyy="0.000561" izz="0.000556" ixy="0.0" iyz="-0.0" ixz="0.0"/>
-    </inertial>
-    <visual>
-      <origin xyz="1.195 0 -1.7" rpy="0 0 3.14"/>
+      <inertia ixx="0.1" ixy="0.0" ixz="0.0" iyy="0.1" iyz="0.0" izz="0.155" />
+    </inertial>
+    <visual>
+      <origin xyz="1.195 0.0 -1.7" rpy="0 0 3.14"/>
       <geometry>
         <mesh filename="file://$(find warehouse_bot)/meshes/mid-360-asm_1.stl" scale="0.001 0.001 0.001"/>
@@ -237,5 +237,5 @@
     </visual>
     <collision>
-      <origin xyz="1.195 0 -1.7" rpy="0 0 3.14"/>
+      <origin xyz="1.195 0.0 -1.7" rpy="0 0 3.14"/>
       <geometry>
         <mesh filename="file://$(find warehouse_bot)/meshes/mid-360-asm_1.stl" scale="0.001 0.001 0.001"/>
@@ -243,5 +243,5 @@
     </collision>
   </link>
-  <link name="laser_frame">
+  <!-- <link name="laser_frame_under">
     <inertial>
       <origin xyz="0 0 0" rpy="0 0 0"/>
@@ -262,5 +262,5 @@
       </geometry>
     </collision>
-  </link>
+  </link>  -->
   <link name="fork_1">
     <inertial>
@@ -270,5 +270,5 @@
     </inertial>
     <visual>
-      <origin xyz="0 0 -0.03" rpy="0 0 0"/>
+      <origin xyz="0.0 0.0 -0.03" rpy="0 0 0"/>
       <geometry>
         <mesh filename="file://$(find warehouse_bot)/meshes/fork_1.stl" scale="0.001 0.001 0.001"/>
@@ -277,5 +277,5 @@
     </visual>
     <collision>
-      <origin xyz="0 0 -0.03" rpy="0 0 0"/>
+      <origin xyz="0.0 0 -0.03" rpy="0 0 0"/>
       <geometry>
         <mesh filename="file://$(find warehouse_bot)/meshes/fork_1.stl" scale="0.001 0.001 0.001"/>
@@ -284,37 +284,39 @@
   </link>
   <joint name="fork_joint" type="fixed">
-    <origin xyz="0 0.0 0.022893" rpy="0 0 0"/>
+    <origin xyz="0.0 0.0 0.022893" rpy="0 0 0"/>
     <parent link="base_link"/>
     <child link="fork_1"/>
   </joint>
   <joint name="left_rs_joint" type="fixed">
-    <origin xyz="-0.46 0.18 0.052" rpy="0 0 3.14"/>
+    <origin xyz="-0.46 0.2 0.052" rpy="0 0 3.14"/>
     <parent link="chassis"/>
     <child link="Intel_Realsense_D435_1"/>
   </joint>
   <joint name="right_rs_joint" type="fixed">
-    <origin xyz="-0.46 -0.18 0.052" rpy="0 0 3.14"/>
+    <origin xyz="-0.46 -0.2 0.052" rpy="0 0 3.14"/>
     <parent link="chassis"/>
     <child link="Intel_Realsense_D435_2"/>
   </joint>
   <joint name="top_rs_joint" type="fixed">
-    <origin xyz="1.0 0 1.76" rpy="0 0.39 3.14"/>
+    <origin xyz="1.0 0.0 1.76" rpy="0 0.39 3.14"/>
     <parent link="chassis"/>
     <child link="Intel_Realsense_D435_3"/>
   </joint>
   <joint name="mid360_joint" type="fixed">
-    <origin xyz="1.175 0 1.68" rpy="0 0 0"/>
+    <origin xyz="1.175 0.0 1.68" rpy="0 0 0"/>
     <parent link="chassis"/>
     <child link="mid-360-asm_1"/>
   </joint>
-  <joint name="16line_lidar_joint" type="fixed">
-    <origin xyz="1.1 0 2.185" rpy="0 0 0"/>
+  <!-- <joint name="16line_lidar_joint" type="fixed">
+    <origin xyz="1.1 0.0 2.25" rpy="0 0 0"/>
     <parent link="chassis"/>
     <child link="line_lidar_1"/>
-  </joint>
-  <joint name="laser_joint" type="fixed">
-    <origin xyz="1.6 0 0.02" rpy="0 0 0"/>
-    <parent link="chassis"/>
-    <child link="laser_frame"/>
-  </joint>
+  </joint> -->
+<!--
+  <joint name="laser_joint1" type="fixed">
+    <origin xyz="1.6 0.0 0.02" rpy="0 0 0"/>
+    <parent link="chassis"/>
+    <child link="laser_frame_under"/>
+  </joint>
+   -->
 </robot>
