Commit message: spawn robot in gazebo warehouse world

File: urdf/gazebo_control.xacro (robot description, xacro)
@@ -5,11 +5,11 @@
             <pose> 0 0 0 0 0 0 </pose>
             <visualize>false</visualize>
-            <update_rate>50</update_rate>
+            <update_rate>10</update_rate>
             <ray>
                 <scan>
                     <horizontal>
                         <samples>360</samples>
-                        <min_angle>-1.57</min_angle>
-                        <max_angle>1.57</max_angle>
+                        <min_angle>-2.2</min_angle>
+                        <max_angle>2.2</max_angle>
                     </horizontal>
                 </scan>

File: urdf/warehouse_bot.xacro (robot description, xacro)
@@ -25,19 +25,19 @@
     <link name="chassis">
       <visual>
-        <origin xyz="0 0 -0.04" rpy="0 0 0"/>
-        <geometry>
-          <mesh filename="file://$(find warehouse_bot)/meshes/chassis.stl" scale="0.002 0.002 0.002"/>
+        <origin xyz="0 0 -0.02" rpy="0 0 0"/>
+        <geometry>
+          <mesh filename="file://$(find warehouse_bot)/meshes/chassis.stl" scale="0.001 0.001 0.001"/>
         </geometry>
         <material name="Orange"/>
       </visual>
       <collision>
-        <origin xyz="0 0 -0.04" rpy="0 0 0"/>
-        <geometry>
-          <mesh filename="file://$(find warehouse_bot)/meshes/chassis.stl" scale="0.002 0.002 0.002"/>
+        <origin xyz="0 0 -0.02" rpy="0 0 0"/>
+        <geometry>
+          <mesh filename="file://$(find warehouse_bot)/meshes/chassis.stl" scale="0.001 0.001 0.001"/>
         </geometry>
       </collision>
       <inertial>
         <origin xyz="0 0 0" rpy="0 0 0" />
-        <mass value="70" />
+        <mass value="45" />
         <inertia ixx="0.126164" ixy="0.0" ixz="0.0" iyy="0.416519" iyz="0.0" izz="0.481014" />
       </inertial>
@@ -52,10 +52,35 @@
       <collision>
         <geometry>
-          <cylinder length="0.08" radius="0.15" />
-        </geometry>
-      </collision>
-      <visual>
-        <geometry>
-          <cylinder length="0.08" radius="0.15" />
+          <cylinder length="0.04" radius="0.075" />
+        </geometry>
+      </collision>
+      <visual>
+        <geometry>
+          <cylinder length="0.04" radius="0.075" />
+        </geometry>
+        <material name="Black" />
+      </visual>
+      <inertial>
+        <mass value="5" />
+        <inertia ixx="0.145833" ixy="0.0" ixz="0.0" iyy="0.145833" iyz="0.0" izz="0.125" />
+      </inertial>
+    </link>
+    <joint name="left_wheel_joint" type="continuous">
+      <origin xyz="0 0.2 0" rpy="-1.57 0 0" />
+      <parent link="chassis" />
+      <child link="left_wheel" />
+      <axis xyz="0 0 1" />
+      <dynamics damping="0.2" />
+    </joint>
+    <!-- right wheel Link -->
+    <link name="right_wheel">
+      <collision>
+        <geometry>
+          <cylinder length="0.04" radius="0.075" />
+        </geometry>
+      </collision>
+      <visual>
+        <geometry>
+          <cylinder length="0.04" radius="0.075" />
         </geometry>
         <material name="Black" />
@@ -66,31 +91,6 @@
       </inertial>
     </link>
-    <joint name="left_wheel_joint" type="continuous">
-      <origin xyz="0 0.4 0" rpy="-1.57 0 0" />
-      <parent link="chassis" />
-      <child link="left_wheel" />
-      <axis xyz="0 0 1" />
-      <dynamics damping="0.2" />
-    </joint>
-    <!-- right wheel Link -->
-    <link name="right_wheel">
-      <collision>
-        <geometry>
-          <cylinder length="0.08" radius="0.15" />
-        </geometry>
-      </collision>
-      <visual>
-        <geometry>
-          <cylinder length="0.08" radius="0.15" />
-        </geometry>
-        <material name="Black" />
-      </visual>
-      <inertial>
-        <mass value="10" />
-        <inertia ixx="0.145833" ixy="0.0" ixz="0.0" iyy="0.145833" iyz="0.0" izz="0.125" />
-      </inertial>
-    </link>
     <joint name="right_wheel_joint" type="continuous">
-      <origin xyz="0 -0.4 0" rpy="-1.57 0 0" />
+      <origin xyz="0 -0.2 0" rpy="-1.57 0 0" />
       <parent link="chassis" />
       <child link="right_wheel" />
@@ -113,5 +113,5 @@
     </link>
     <joint name="steering_joint" type="continuous">
-      <origin xyz="2.2 0 0" rpy="0 0 0" />
+      <origin xyz="1.1 0 0" rpy="0 0 0" />
       <parent link="chassis" />
       <child link="steering_link" />
@@ -122,5 +122,5 @@
       <visual>
         <geometry>
-          <cylinder length="0.08" radius="0.15" />
+          <cylinder length="0.04" radius="0.075" />
         </geometry>
         <material name="Black" />
@@ -133,5 +133,5 @@
       <collision>
         <geometry>
-          <cylinder length="0.08" radius="0.15" />
+          <cylinder length="0.04" radius="0.075" />
         </geometry>
       </collision>
@@ -153,5 +153,5 @@
       <origin xyz="0.92 0.38 0.12" rpy="3.14 0 0"/>
       <geometry>
-        <mesh filename="file://$(find warehouse_bot)/meshes/Intel_Realsense_D435_1.stl" scale="0.002 0.002 0.002"/>
+        <mesh filename="file://$(find warehouse_bot)/meshes/Intel_Realsense_D435_1.stl" scale="0.001 0.001 0.001"/>
       </geometry>
       <material name="silver"/>
@@ -160,5 +160,5 @@
       <origin xyz="0.92 0.38 0.12" rpy="3.14 0 0"/>
       <geometry>
-        <mesh filename="file://$(find warehouse_bot)/meshes/Intel_Realsense_D435_1.stl" scale="0.002 0.002 0.002"/>
+        <mesh filename="file://$(find warehouse_bot)/meshes/Intel_Realsense_D435_1.stl" scale="0.001 0.001 0.001"/>
       </geometry>
     </collision>
@@ -173,5 +173,5 @@
       <origin xyz="0.92 -0.38 0.12" rpy="3.14 0 0"/>
       <geometry>
-        <mesh filename="file://$(find warehouse_bot)/meshes/Intel_Realsense_D435_2.stl" scale="0.002 0.002 0.002"/>
+        <mesh filename="file://$(find warehouse_bot)/meshes/Intel_Realsense_D435_2.stl" scale="0.001 0.001 0.001"/>
       </geometry>
       <material name="silver"/>
@@ -180,5 +180,5 @@
       <origin xyz="0.92 -0.38 0.12" rpy="3.14 0 0"/>
       <geometry>
-        <mesh filename="file://$(find warehouse_bot)/meshes/Intel_Realsense_D435_2.stl" scale="0.002 0.002 0.002"/>
+        <mesh filename="file://$(find warehouse_bot)/meshes/Intel_Realsense_D435_2.stl" scale="0.001 0.001 0.001"/>
       </geometry>
     </collision>
@@ -193,5 +193,5 @@
       <origin xyz="-2.0 0 -3.54" rpy="0 0 0"/>
       <geometry>
-        <mesh filename="file://$(find warehouse_bot)/meshes/Intel_Realsense_D435_3.stl" scale="0.002 0.002 0.002"/>
+        <mesh filename="file://$(find warehouse_bot)/meshes/Intel_Realsense_D435_3.stl" scale="0.001 0.001 0.001"/>
       </geometry>
       <material name="silver"/>
@@ -200,5 +200,5 @@
       <origin xyz="-2.0 0 -3.54" rpy="0 0 0"/>
       <geometry>
-        <mesh filename="file://$(find warehouse_bot)/meshes/Intel_Realsense_D435_3.stl" scale="0.002 0.002 0.002"/>
+        <mesh filename="file://$(find warehouse_bot)/meshes/Intel_Realsense_D435_3.stl" scale="0.001 0.001 0.001"/>
       </geometry>
     </collision>
@@ -213,5 +213,5 @@
       <origin xyz="-2.2 0 4.37" rpy="3.14 0 0"/>
       <geometry>
-        <mesh filename="file://$(find warehouse_bot)/meshes/16line_lidar_1.stl" scale="0.002 0.002 0.002"/>
+        <mesh filename="file://$(find warehouse_bot)/meshes/16line_lidar_1.stl" scale="0.001 0.001 0.001"/>
       </geometry>
       <material name="silver"/>
@@ -220,5 +220,5 @@
       <origin xyz="-2.2 0 4.37" rpy="3.14 0 0"/>
       <geometry>
-        <mesh filename="file://$(find warehouse_bot)/meshes/16line_lidar_1.stl" scale="0.002 0.002 0.002"/>
+        <mesh filename="file://$(find warehouse_bot)/meshes/16line_lidar_1.stl" scale="0.001 0.001 0.001"/>
       </geometry>
     </collision>
@@ -233,5 +233,5 @@
       <origin xyz="2.39 0 -3.4" rpy="0 0 3.14"/>
       <geometry>
-        <mesh filename="file://$(find warehouse_bot)/meshes/mid-360-asm_1.stl" scale="0.002 0.002 0.002"/>
+        <mesh filename="file://$(find warehouse_bot)/meshes/mid-360-asm_1.stl" scale="0.001 0.001 0.001"/>
       </geometry>
       <material name="silver"/>
@@ -240,5 +240,5 @@
       <origin xyz="2.39 0 -3.4" rpy="0 0 3.14"/>
       <geometry>
-        <mesh filename="file://$(find warehouse_bot)/meshes/mid-360-asm_1.stl" scale="0.002 0.002 0.002"/>
+        <mesh filename="file://$(find warehouse_bot)/meshes/mid-360-asm_1.stl" scale="0.001 0.001 0.001"/>
       </geometry>
     </collision>
@@ -251,14 +251,14 @@
     </inertial>
     <visual>
-      <origin xyz="-2.95 0 0.01" rpy="3.14 0 0"/>
-      <geometry>
-        <mesh filename="file://$(find warehouse_bot)/meshes/1line_lidar_1.stl" scale="0.002 0.002 0.002"/>
-      </geometry>
-      <material name="silver"/>
-    </visual>
-    <collision>
-      <origin xyz="-2.95 0 0.01" rpy="3.14 0 0"/>
-      <geometry>
-        <mesh filename="file://$(find warehouse_bot)/meshes/1line_lidar_1.stl" scale="0.002 0.002 0.002"/>
+      <origin xyz="-1.475 0 0.005" rpy="3.14 0 0"/>
+      <geometry>
+        <mesh filename="file://$(find warehouse_bot)/meshes/1line_lidar_1.stl" scale="0.001 0.001 0.001"/>
+      </geometry>
+      <material name="silver"/>
+    </visual>
+    <collision>
+      <origin xyz="-1.475 0 0.005" rpy="3.14 0 0"/>
+      <geometry>
+        <mesh filename="file://$(find warehouse_bot)/meshes/1line_lidar_1.stl" scale="0.001 0.001 0.001"/>
       </geometry>
     </collision>
@@ -289,6 +289,6 @@
     <child link="16line_lidar_1"/>
   </joint> -->
-  <joint name="laser_frame_joint" type="fixed">
-    <origin xyz="3.2 0 0.04" rpy="0 0 0"/>
+  <joint name="laser_joint" type="fixed">
+    <origin xyz="1.6 0 0.02" rpy="0 0 0"/>
     <parent link="chassis"/>
     <child link="laser_frame"/>

Commit message: fix bags with cameras and controller, can start in world

File: urdf/gazebo_control.xacro (robot description, xacro)
@@ -1,5 +1,5 @@
 <?xml version="1.0"?>
 <robot>
-    <gazebo reference="laser_frame">
+    <gazebo reference="line_lidar_1">
         <sensor name="laser" type="ray">
             <pose> 0 0 0 0 0 0 </pose>
@@ -10,6 +10,6 @@
                     <horizontal>
                         <samples>360</samples>
-                        <min_angle>-2.2</min_angle>
-                        <max_angle>2.2</max_angle>
+                        <min_angle>-3.14</min_angle>
+                        <max_angle>3.14</max_angle>
                     </horizontal>
                 </scan>
@@ -24,5 +24,5 @@
                 </ros>
                 <output_type>sensor_msgs/LaserScan</output_type>
-                <frame_name>laser_frame</frame_name>
+                <frame_name>line_lidar_1</frame_name>
             </plugin>
         </sensor>

File: urdf/robot.urdf.xacro (robot description, xacro)
@@ -2,5 +2,5 @@
 <robot xmlns:xacro="http://www.ros.org/wiki/xacro"  name="robot">
     <xacro:include filename="warehouse_bot.xacro" />
+    <xacro:include filename="gazebo_control.xacro" />
     <xacro:include filename="ros2_control.xacro" />
-    <xacro:include filename="gazebo_control.xacro" />
 </robot>

File: urdf/warehouse_bot.xacro (robot description, xacro)
@@ -39,6 +39,6 @@
       <inertial>
         <origin xyz="0 0 0" rpy="0 0 0" />
-        <mass value="45" />
-        <inertia ixx="0.126164" ixy="0.0" ixz="0.0" iyy="0.416519" iyz="0.0" izz="0.481014" />
+        <mass value="70" />
+        <inertia ixx="2.5" ixy="0.0" ixz="0.0" iyy="1.5" iyz="0.0" izz="3.7" />
       </inertial>
     </link>
@@ -62,5 +62,5 @@
       </visual>
       <inertial>
-        <mass value="5" />
+        <mass value="10" />
         <inertia ixx="0.145833" ixy="0.0" ixz="0.0" iyy="0.145833" iyz="0.0" izz="0.125" />
       </inertial>
@@ -108,6 +108,6 @@
       <inertial>
         <origin xyz="0 0 0" rpy="0 0 0" />
-        <mass value="0.005" />
-        <inertia ixx="0.1" ixy="0.0" ixz="0.0" iyy="0.1" iyz="0.0" izz="0.1" />
+        <mass value="10" />
+        <inertia ixx="0.01" ixy="0.0" ixz="0.0" iyy="0.01" iyz="0.0" izz="0.01" />
       </inertial>
     </link>
@@ -129,5 +129,5 @@
         <origin xyz="0 0 0" rpy="0 0 0" />
         <mass value="20" />
-        <inertia ixx="1" ixy="0" ixz="0" iyy="1" iyz="0" izz="1" />
+        <inertia ixx="0.01" ixy="0" ixz="0" iyy="0.01" iyz="0" izz="0.01" />
       </inertial>
       <collision>
@@ -143,6 +143,5 @@
       <axis xyz="0 0 1" />
     </joint>
-<!--
-    <link name="Intel_Realsense_D435_1">
+  <link name="Intel_Realsense_D435_1">
     <inertial>
       <origin xyz="0 0 0" rpy="0 0 0"/>
@@ -151,5 +150,5 @@
     </inertial>
     <visual>
-      <origin xyz="0.92 0.38 0.12" rpy="3.14 0 0"/>
+      <origin xyz="0.46 0.19 0.06" rpy="3.14 0 0"/>
       <geometry>
         <mesh filename="file://$(find warehouse_bot)/meshes/Intel_Realsense_D435_1.stl" scale="0.001 0.001 0.001"/>
@@ -158,5 +157,5 @@
     </visual>
     <collision>
-      <origin xyz="0.92 0.38 0.12" rpy="3.14 0 0"/>
+      <origin xyz="0.46 0.19 0.06" rpy="3.14 0 0"/>
       <geometry>
         <mesh filename="file://$(find warehouse_bot)/meshes/Intel_Realsense_D435_1.stl" scale="0.001 0.001 0.001"/>
@@ -171,5 +170,5 @@
     </inertial>
     <visual>
-      <origin xyz="0.92 -0.38 0.12" rpy="3.14 0 0"/>
+      <origin xyz="0.46 -0.19 0.06" rpy="3.14 0 0"/>
       <geometry>
         <mesh filename="file://$(find warehouse_bot)/meshes/Intel_Realsense_D435_2.stl" scale="0.001 0.001 0.001"/>
@@ -178,5 +177,5 @@
     </visual>
     <collision>
-      <origin xyz="0.92 -0.38 0.12" rpy="3.14 0 0"/>
+      <origin xyz="0.46 -0.19 0.06" rpy="3.14 0 0"/>
       <geometry>
         <mesh filename="file://$(find warehouse_bot)/meshes/Intel_Realsense_D435_2.stl" scale="0.001 0.001 0.001"/>
@@ -191,5 +190,5 @@
     </inertial>
     <visual>
-      <origin xyz="-2.0 0 -3.54" rpy="0 0 0"/>
+      <origin xyz="-1.0 0 -1.77" rpy="0 0 0"/>
       <geometry>
         <mesh filename="file://$(find warehouse_bot)/meshes/Intel_Realsense_D435_3.stl" scale="0.001 0.001 0.001"/>
@@ -198,5 +197,5 @@
     </visual>
     <collision>
-      <origin xyz="-2.0 0 -3.54" rpy="0 0 0"/>
+      <origin xyz="-1.0 0 -1.77" rpy="0 0 0"/>
       <geometry>
         <mesh filename="file://$(find warehouse_bot)/meshes/Intel_Realsense_D435_3.stl" scale="0.001 0.001 0.001"/>
@@ -204,12 +203,12 @@
     </collision>
   </link>
-  <link name="16line_lidar_1">
-    <inertial>
-      <origin xyz="0 0 0" rpy="0 0 0"/>
-      <mass value="0.01"/>
-      <inertia ixx="0.008817" iyy="0.008817" izz="0.007464" ixy="-0.0" iyz="0.0" ixz="-0.0"/>
-    </inertial>
-    <visual>
-      <origin xyz="-2.2 0 4.37" rpy="3.14 0 0"/>
+  <link name="line_lidar_1">
+    <inertial>
+      <origin xyz="0 0 0" rpy="0 0 0"/>
+      <mass value="1"/>
+      <inertia ixx="0.00068" iyy="0.00068" izz="0.000389" ixy="0.0" iyz="-0.0" ixz="-0.0"/>
+    </inertial>
+    <visual>
+      <origin xyz="-1.1 0 2.29" rpy="3.14 0 0"/>
       <geometry>
         <mesh filename="file://$(find warehouse_bot)/meshes/16line_lidar_1.stl" scale="0.001 0.001 0.001"/>
@@ -218,5 +217,5 @@
     </visual>
     <collision>
-      <origin xyz="-2.2 0 4.37" rpy="3.14 0 0"/>
+      <origin xyz="-1.1 0 2.29" rpy="3.14 0 0"/>
       <geometry>
         <mesh filename="file://$(find warehouse_bot)/meshes/16line_lidar_1.stl" scale="0.001 0.001 0.001"/>
@@ -231,5 +230,5 @@
     </inertial>
     <visual>
-      <origin xyz="2.39 0 -3.4" rpy="0 0 3.14"/>
+      <origin xyz="1.195 0 -1.7" rpy="0 0 3.14"/>
       <geometry>
         <mesh filename="file://$(find warehouse_bot)/meshes/mid-360-asm_1.stl" scale="0.001 0.001 0.001"/>
@@ -238,14 +237,14 @@
     </visual>
     <collision>
-      <origin xyz="2.39 0 -3.4" rpy="0 0 3.14"/>
+      <origin xyz="1.195 0 -1.7" rpy="0 0 3.14"/>
       <geometry>
         <mesh filename="file://$(find warehouse_bot)/meshes/mid-360-asm_1.stl" scale="0.001 0.001 0.001"/>
       </geometry>
     </collision>
-  </link> -->
+  </link>
   <link name="laser_frame">
     <inertial>
       <origin xyz="0 0 0" rpy="0 0 0"/>
-      <mass value="0.01"/>
+      <mass value="10"/>
       <inertia ixx="0.00068" iyy="0.00068" izz="0.000389" ixy="0.0" iyz="-0.0" ixz="-0.0"/>
     </inertial>
@@ -264,29 +263,54 @@
     </collision>
   </link>
-  <!-- <joint name="left_rs_joint" type="fixed">
-    <origin xyz="-0.3 0.4 0.05" rpy="0 0 3.14"/>
+  <link name="fork_1">
+    <inertial>
+      <origin xyz="0 0 0" rpy="0 0 0"/>
+      <mass value="10"/>
+      <inertia ixx="0.1" ixy="0.0" ixz="0.0" iyy="0.1" iyz="0.0" izz="0.155" />
+    </inertial>
+    <visual>
+      <origin xyz="0 0 -0.03" rpy="0 0 0"/>
+      <geometry>
+        <mesh filename="file://$(find warehouse_bot)/meshes/fork_1.stl" scale="0.001 0.001 0.001"/>
+      </geometry>
+      <material name="silver"/>
+    </visual>
+    <collision>
+      <origin xyz="0 0 -0.03" rpy="0 0 0"/>
+      <geometry>
+        <mesh filename="file://$(find warehouse_bot)/meshes/fork_1.stl" scale="0.001 0.001 0.001"/>
+      </geometry>
+    </collision>
+  </link>
+  <joint name="fork_joint" type="fixed">
+    <origin xyz="0 0.0 0.022893" rpy="0 0 0"/>
+    <parent link="base_link"/>
+    <child link="fork_1"/>
+  </joint>
+  <joint name="left_rs_joint" type="fixed">
+    <origin xyz="-0.46 0.18 0.052" rpy="0 0 3.14"/>
     <parent link="chassis"/>
     <child link="Intel_Realsense_D435_1"/>
   </joint>
   <joint name="right_rs_joint" type="fixed">
-    <origin xyz="-0.3 -0.4 0.05" rpy="0 0 3.14"/>
+    <origin xyz="-0.46 -0.18 0.052" rpy="0 0 3.14"/>
     <parent link="chassis"/>
     <child link="Intel_Realsense_D435_2"/>
   </joint>
   <joint name="top_rs_joint" type="fixed">
-    <origin xyz="2.0 0 3.52" rpy="0 0.39 3.14"/>
+    <origin xyz="1.0 0 1.76" rpy="0 0.39 3.14"/>
     <parent link="chassis"/>
     <child link="Intel_Realsense_D435_3"/>
   </joint>
   <joint name="mid360_joint" type="fixed">
-    <origin xyz="2.35 0 3.3404" rpy="0 0 0"/>
+    <origin xyz="1.175 0 1.68" rpy="0 0 0"/>
     <parent link="chassis"/>
     <child link="mid-360-asm_1"/>
-  </joint>  -->
-  <!-- <joint name="16line_lidar_joint" type="fixed">
-    <origin xyz="2.2 0 4.37" rpy="0 0 0"/>
-    <parent link="chassis"/>
-    <child link="16line_lidar_1"/>
-  </joint> -->
+  </joint>
+  <joint name="16line_lidar_joint" type="fixed">
+    <origin xyz="1.1 0 2.185" rpy="0 0 0"/>
+    <parent link="chassis"/>
+    <child link="line_lidar_1"/>
+  </joint>
   <joint name="laser_joint" type="fixed">
     <origin xyz="1.6 0 0.02" rpy="0 0 0"/>

Commit message: fix bugs with launch, and up velocity, nav2 ok

File: urdf/gazebo_control.xacro (robot description, xacro)
@@ -5,5 +5,5 @@
             <pose> 0 0 0 0 0 0 </pose>
             <visualize>false</visualize>
-            <update_rate>10</update_rate>
+            <update_rate>100</update_rate>
             <ray>
                 <scan>

File: urdf/warehouse_bot.xacro (robot description, xacro)
@@ -108,5 +108,5 @@
       <inertial>
         <origin xyz="0 0 0" rpy="0 0 0" />
-        <mass value="10" />
+        <mass value="40" />
         <inertia ixx="0.01" ixy="0.0" ixz="0.0" iyy="0.01" iyz="0.0" izz="0.01" />
       </inertial>

Commit message: fix bugs

File: urdf/gazebo_control.xacro (robot description, xacro)
@@ -5,5 +5,5 @@
             <pose> 0 0 0 0 0 0 </pose>
             <visualize>false</visualize>
-            <update_rate>100</update_rate>
+            <update_rate>10</update_rate>
             <ray>
                 <scan>
@@ -16,5 +16,5 @@
                 <range>
                     <min>0.3</min>
-                    <max>20</max>
+                    <max>150</max>
                 </range>
             </ray>

File: urdf/lidar.xacro (robot description, xacro)
@@ -11,5 +11,4 @@
                 <cylinder radius="0.05" length="0.04"/>
             </geometry>
-            <material name="black"/>
         </visual>
         <visual>
@@ -18,5 +17,4 @@
                 <cylinder radius="0.01" length="0.2"/>
             </geometry>
-            <material name="black"/>
         </visual>
         <collision>
@@ -32,5 +30,4 @@
     </link>
     <gazebo reference="laser_frame">
-        <material>Gazebo/Black</material>
         <sensor name="laser" type="ray">
             <pose> 0 0 0 0 0 0 </pose>

File: urdf/robot.urdf.xacro (robot description, xacro)
@@ -3,4 +3,4 @@
     <xacro:include filename="warehouse_bot.xacro" />
     <xacro:include filename="ros2_control.xacro" />
-    <xacro:include filename="lidar.xacro" />
+    <xacro:include filename="gazebo_control.xacro" />
 </robot>

File: urdf/warehouse_bot.xacro (robot description, xacro)
@@ -143,5 +143,5 @@
       <axis xyz="0 0 1" />
     </joint>
-  <link name="Intel_Realsense_D435_1">
+  <!-- <link name="Intel_Realsense_D435_1">
     <inertial>
       <origin xyz="0 0 0" rpy="0 0 0"/>
@@ -199,6 +199,6 @@
       </geometry>
     </collision>
-  </link>
-  <!-- <link name="line_lidar_1">
+  </link> -->
+  <link name="line_lidar_1">
     <inertial>
       <origin xyz="0 0 0" rpy="0 0 0"/>
@@ -218,5 +218,6 @@
       </geometry>
     </collision>
-  </link> -->
+  </link>
+<!--
   <link name="mid-360-asm_1">
     <inertial>
@@ -237,5 +238,5 @@
       </geometry>
     </collision>
-  </link>
+  </link> -->
   <!-- <link name="laser_frame_under">
     <inertial>
@@ -281,5 +282,5 @@
     <child link="fork_1"/>
   </joint>
-  <joint name="left_rs_joint" type="fixed">
+  <!-- <joint name="left_rs_joint" type="fixed">
     <origin xyz="-0.46 0.2 0.052" rpy="0 0 3.14"/>
     <parent link="chassis"/>
@@ -300,10 +301,10 @@
     <parent link="chassis"/>
     <child link="mid-360-asm_1"/>
-  </joint>
-  <!-- <joint name="16line_lidar_joint" type="fixed">
+  </joint>  -->
+  <joint name="16line_lidar_joint" type="fixed">
     <origin xyz="1.1 0.0 2.25" rpy="0 0 0"/>
     <parent link="chassis"/>
     <child link="line_lidar_1"/>
-  </joint> -->
+  </joint>
 <!--
   <joint name="laser_joint1" type="fixed">
