Commit message: 2d branch

File: warehouse_bot/urdf/robot.urdf.xacro (robot description, xacro)
@@ -4,5 +4,4 @@
     <xacro:include filename="$(find warehouse_bot)/urdf/_d435.urdf1.xacro" />
     <xacro:include filename="$(find warehouse_bot)/urdf/_d435.urdf3.xacro" />
-    <xacro:include filename="$(find ros2_livox_simulation)/urdf/mid360.xacro" />
     <xacro:include filename="warehouse_bot.xacro" />
     <xacro:include filename="ros2_control.xacro" />

File: warehouse_bot/urdf/warehouse_bot.xacro (robot description, xacro)
@@ -233,9 +233,4 @@
     <origin xyz="1.0 0.0 1.77" rpy="0 2.2 3.14" />
   </xacro:sensor_d435_3>
-  <!-- <joint name="mid360_joint" type="fixed">
-    <origin xyz="1.175 0.0 1.68" rpy="0 0 0"/>
-    <parent link="chassis"/>
-    <child link="mid-360-asm_1"/>
-  </joint>  -->
   <joint name="16line_lidar_joint" type="fixed">
     <origin xyz="1.1 0.0 2.24" rpy="0 0 0"/>
@@ -248,6 +243,3 @@
     <child link="laser_frame_under"/>
   </joint>
-  <xacro:mid360 name="livox" parent="base_link" topic="mid360">
-    <origin xyz="1.175 0.0 1.67" rpy="3.14 0 0"/>
-  </xacro:mid360>
 </robot>
