Commit message: fix controller and mppi

File: warehouse_bot/urdf/warehouse_bot.xacro (robot description, xacro)
@@ -60,5 +60,5 @@
       <child link="front_steering_hinge_link" />
       <axis xyz="0 0 1" />
-      <limit lower="-0.7853" upper="0.7853" effort="10" velocity="100" />
+      <limit lower="-1.57" upper="1.57" effort="10" velocity="100" />
     </joint>
     <!-- Front Wheel Link -->
