Commit message: update nav2

File: warehouse_bot/urdf/gazebo_control.xacro (robot description, xacro)
@@ -37,5 +37,5 @@
             <pose> 0 0 0 0 0 0 </pose>
             <always_on>true</always_on>
-            <visualize>true</visualize>
+            <visualize>false</visualize>
             <update_rate>10</update_rate>
             <ray>
@@ -49,10 +49,10 @@
                 <range>
                     <min>0.3</min>
-                    <max>150</max>
+                    <max>15.0</max>
                 </range>
             </ray>
             <plugin name="laser_controller1" filename="libgazebo_ros_ray_sensor.so">
                 <ros>
-                    <argument>~/out:=scan</argument>
+                    <remapping>~/out:=scan</remapping>
                 </ros>
                 <output_type>sensor_msgs/LaserScan</output_type>
@@ -70,16 +70,16 @@
                     <horizontal>
                         <samples>360</samples>
-                        <min_angle>-1.4</min_angle>
-                        <max_angle>1.4</max_angle>
+                        <min_angle>-2.4</min_angle>
+                        <max_angle>2.4</max_angle>
                     </horizontal>
                 </scan>
                 <range>
                     <min>0.3</min>
-                    <max>150</max>
+                    <max>15.0</max>
                 </range>
             </ray>
             <plugin name="laser_controller2" filename="libgazebo_ros_ray_sensor.so">
                 <ros>
-                    <argument>~/out:=scan2</argument>
+                    <remapping>~/out:=scan2</remapping>
                 </ros>
                 <output_type>sensor_msgs/LaserScan</output_type>

File: warehouse_bot/urdf/warehouse_bot.xacro (robot description, xacro)
@@ -38,5 +38,5 @@
         <origin xyz="0 0 0" rpy="0 0 0" />
         <mass value="70" />
-        <inertia ixx="0.126164" ixy="0.0" ixz="0.0" iyy="0.416519" iyz="0.0" izz="0.481014" />
+        <inertia ixx="0.011642" iyy="0.035651" izz="0.038255" ixy="0.000148" iyz="-9.3e-05" ixz="0.000342"/>
       </inertial>
     </link>

Commit message: add 16line_lidar add

File: warehouse_bot/urdf/gazebo_control.xacro (robot description, xacro)
@@ -33,5 +33,5 @@
         <material>Gazebo/Black</material>
     </gazebo>
-    <gazebo reference="line_lidar_1">
+    <!-- <gazebo reference="line_lidar_1">
         <sensor name="laser1" type="ray">
             <pose> 0 0 0 0 0 0 </pose>
@@ -60,5 +60,5 @@
             </plugin>
         </sensor>
-    </gazebo>
+    </gazebo> -->
     <gazebo reference="laser_frame_under">
         <sensor name="laser2" type="ray">

File: warehouse_bot/urdf/robot.urdf.xacro (robot description, xacro)
@@ -5,4 +5,5 @@
     <xacro:include filename="$(find warehouse_bot)/urdf/_d435.urdf1.xacro" />
     <xacro:include filename="$(find warehouse_bot)/urdf/_d435.urdf3.xacro" /> -->
+    <xacro:include filename="$(find robosense_description)/urdf/RS-16.urdf.xacro"/>
     <xacro:include filename="$(find warehouse_bot)/urdf/materials.xacro" />
     <xacro:include filename="$(find warehouse_bot)/urdf/macros.xacro" />

File: warehouse_bot/urdf/warehouse_bot.xacro (robot description, xacro)
@@ -1,4 +1,6 @@
 <?xml version="1.0"?>
 <robot name="robot_1" xmlns:xacro="http://ros.org/wiki/xacro">
+    <xacro:arg name="gpu" default="false"/>
+    <xacro:property name="gpu" value="$(arg gpu)" />
     <material name="Black">
       <color rgba="0 0 0 1" />
@@ -155,5 +157,5 @@
     <child link="imu_link"/>
   </joint>
-  <link name="line_lidar_1">
+  <!-- <link name="line_lidar_1">
     <inertial>
       <origin xyz="0 0 0" rpy="0 0 0"/>
@@ -173,5 +175,5 @@
       </geometry>
     </collision>
-  </link>
+  </link> -->
   <link name="laser_frame_under">
     <inertial>
@@ -226,9 +228,9 @@
     <origin xyz="1.0 0.0 1.77" rpy="0 2.2 3.14" />
   </xacro:sensor_d435_3>   -->
-  <joint name="16line_lidar_joint" type="fixed">
+  <!-- <joint name="16line_lidar_joint" type="fixed">
     <origin xyz="1.1 0.0 2.24" rpy="0 0 0"/>
     <parent link="chassis"/>
     <child link="line_lidar_1"/>
-  </joint>
+  </joint> -->
   <joint name="laser_joint1" type="fixed">
     <origin xyz="1.6 0.0 0.02" rpy="0 0 0"/>
@@ -236,4 +238,7 @@
     <child link="laser_frame_under"/>
   </joint>
+  <xacro:RS-16 parent="chassis" name="robosense" topic="/rs_points" hz="20" samples="360" gpu="${gpu}">
+    <origin xyz="1.1 0.0 2.24" rpy="0 0 0" />
+  </xacro:RS-16>
   <!-- <xacro:mid360 name="livox" parent="chassis" topic="mid360">
     <origin xyz="1.175 0.0 1.67" rpy="3.14 0 0"/>
