Commit message: localization from namespace

File: warehouse_bot/urdf/gazebo_robots.xacro (robot description, xacro)
@@ -33,5 +33,5 @@
         <material>Gazebo/Black</material>
     </gazebo>
-    <gazebo reference="$(arg robot_name)_line_lidar_1">
+    <!-- <gazebo reference="$(arg robot_name)_line_lidar_1">
         <sensor name="laser1" type="ray">
             <pose> 0 0 0 0 0 0 </pose>
@@ -61,5 +61,5 @@
             </plugin>
         </sensor>
-    </gazebo>
+    </gazebo> -->
     <gazebo reference="$(arg robot_name)_laser_frame_under">
         <sensor name="laser2" type="ray">
@@ -83,5 +83,5 @@
                 <ros>
                     <namespace>$(arg robot_name)</namespace>
-                    <argument>~/out:=scan2</argument>
+                    <argument>~/out:=scan</argument>
                 </ros>
                 <output_type>sensor_msgs/LaserScan</output_type>

File: warehouse_bot/urdf/robots.urdf.xacro (robot description, xacro)
@@ -158,5 +158,5 @@
         <child link="$(arg robot_name)_imu_link"/>
     </joint>
-    <link name="$(arg robot_name)_line_lidar_1">
+    <!-- <link name="$(arg robot_name)_line_lidar_1">
         <inertial>
             <origin xyz="0 0 0" rpy="0 0 0"/>
@@ -176,5 +176,5 @@
             </geometry>
         </collision>
-    </link>
+    </link> -->
     <link name="$(arg robot_name)_laser_frame_under">
         <inertial>
@@ -220,9 +220,9 @@
         <child link="$(arg robot_name)_fork_1"/>
     </joint>
-    <joint name="$(arg robot_name)_16line_lidar_joint" type="fixed">
+    <!-- <joint name="$(arg robot_name)_16line_lidar_joint" type="fixed">
         <origin xyz="1.1 0.0 2.24" rpy="0 0 0"/>
         <parent link="$(arg robot_name)_chassis"/>
         <child link="$(arg robot_name)_line_lidar_1"/>
-    </joint>
+    </joint> -->
     <joint name="$(arg robot_name)_laser_joint1" type="fixed">
         <origin xyz="1.6 0.0 0.02" rpy="0 0 0"/>

Commit message: rmf visualzed robot_1

File: warehouse_bot/urdf/gazebo_robots.xacro (robot description, xacro)
@@ -1,116 +1,119 @@
 <?xml version="1.0"?>
-<robot name="$(arg robot_name)" xmlns:xacro="http://ros.org/wiki/xacro">
-    <!-- Gazebo references -->
-    <gazebo reference="$(arg robot_name)_chassis">
-        <mu1 value="0.0" />
-        <mu2 value="0.0" />
-        <kp value="10000000.0" />
-        <kd value="1.0" />
-        <material>Gazebo/Grey</material>
-    </gazebo>
-    <gazebo reference="$(arg robot_name)_front_wheel_link">
-        <mu1 value="1.0" />
-        <mu2 value="1.0" />
-        <kp value="10000000.0" />
-        <kd value="1.0" />
-        <fdir1 value="0 0 1" />
-        <material>Gazebo/Black</material>
-    </gazebo>
-    <gazebo reference="$(arg robot_name)_lr_wheel_link">
-        <mu1 value="1.0" />
-        <mu2 value="1.0" />
-        <kp value="10000000.0" />
-        <kd value="1.0" />
-        <fdir1 value="1 0 0" />
-        <material>Gazebo/Black</material>
-    </gazebo>
-    <gazebo reference="$(arg robot_name)_rr_wheel_link">
-        <mu1 value="1.0" />
-        <mu2 value="1.0" />
-        <kp value="10000000.0" />
-        <kd value="1.0" />
-        <fdir1 value="1 0 0" />
-        <material>Gazebo/Black</material>
-    </gazebo>
-    <!-- <gazebo reference="$(arg robot_name)_line_lidar_1">
-        <sensor name="laser1" type="ray">
-            <pose> 0 0 0 0 0 0 </pose>
-            <always_on>true</always_on>
-            <visualize>true</visualize>
-            <update_rate>10</update_rate>
-            <ray>
-                <scan>
-                    <horizontal>
-                        <samples>360</samples>
-                        <min_angle>-3.14</min_angle>
-                        <max_angle>3.14</max_angle>
-                    </horizontal>
-                </scan>
-                <range>
-                    <min>0.3</min>
-                    <max>150</max>
-                </range>
-            </ray>
-            <plugin name="laser_controller1" filename="libgazebo_ros_ray_sensor.so">
-                <ros>
-                    <namespace>$(arg robot_name)</namespace>
-                    <argument>~/out:=scan</argument>
-                </ros>
-                <output_type>sensor_msgs/LaserScan</output_type>
-                <frame_name>$(arg robot_name)_line_lidar_1</frame_name>
-            </plugin>
-        </sensor>
-    </gazebo> -->
-    <gazebo reference="$(arg robot_name)_laser_frame_under">
-        <sensor name="laser2" type="ray">
-            <pose> 0 0 0 0 0 0 </pose>
-            <visualize>true</visualize>
-            <update_rate>10</update_rate>
-            <ray>
-                <scan>
-                    <horizontal>
-                        <samples>360</samples>
-                        <min_angle>-1.4</min_angle>
-                        <max_angle>1.4</max_angle>
-                    </horizontal>
-                </scan>
-                <range>
-                    <min>0.3</min>
-                    <max>150</max>
-                </range>
-            </ray>
-            <plugin name="laser_controller2" filename="libgazebo_ros_ray_sensor.so">
-                <ros>
-                    <namespace>$(arg robot_name)</namespace>
-                    <argument>~/out:=scan</argument>
-                </ros>
-                <output_type>sensor_msgs/LaserScan</output_type>
-                <frame_name>$(arg robot_name)_laser_frame_under</frame_name>
-            </plugin>
-        </sensor>
-    </gazebo>
-    <gazebo reference="$(arg robot_name)_imu_link">
-        <gravity>true</gravity>
-        <sensor name="imu_sensor" type="imu">
-            <always_on>true</always_on>
-            <update_rate>100</update_rate>
-            <visualize>true</visualize>
-            <topic>imu</topic>
-            <plugin filename="libgazebo_ros_imu_sensor.so" name="imu_plugin">
-                <topicName>imu</topicName>
-                <bodyName>$(arg robot_name)_imu_link</bodyName>
-                <updateRateHZ>100.0</updateRateHZ>
-                <!-- <gaussianNoise>0.0</gaussianNoise> -->
-                <xyzOffset>0 0 0</xyzOffset>
-                <rpyOffset>0 0 0</rpyOffset>
-                <frameName>$(arg robot_name)_imu_link</frameName>
-                <initialOrientationAsReference>false</initialOrientationAsReference>
-                <ros>
-                    <namespace>$(arg robot_name)/imu</namespace>
-                    <remapping>~/out:=data</remapping>
-                </ros>
-            </plugin>
-            <pose>0 0 0 0 0 0</pose>
-        </sensor>
-    </gazebo>
+<robot xmlns:xacro="http://ros.org/wiki/xacro">
+    <!-- Define a macro that accepts robot_name as a parameter -->
+    <xacro:macro name="robot_gazebo_plugins" params="robot_name">
+        <!-- Gazebo references -->
+        <gazebo reference="${robot_name}_chassis">
+            <mu1 value="0.0" />
+            <mu2 value="0.0" />
+            <kp value="10000000.0" />
+            <kd value="1.0" />
+            <material>Gazebo/Grey</material>
+        </gazebo>
+        <gazebo reference="${robot_name}_front_wheel_link">
+            <mu1 value="1.0" />
+            <mu2 value="1.0" />
+            <kp value="10000000.0" />
+            <kd value="1.0" />
+            <fdir1 value="0 0 1" />
+            <material>Gazebo/Black</material>
+        </gazebo>
+        <gazebo reference="${robot_name}_lr_wheel_link">
+            <mu1 value="1.0" />
+            <mu2 value="1.0" />
+            <kp value="10000000.0" />
+            <kd value="1.0" />
+            <fdir1 value="1 0 0" />
+            <material>Gazebo/Black</material>
+        </gazebo>
+        <gazebo reference="${robot_name}_rr_wheel_link">
+            <mu1 value="1.0" />
+            <mu2 value="1.0" />
+            <kp value="10000000.0" />
+            <kd value="1.0" />
+            <fdir1 value="1 0 0" />
+            <material>Gazebo/Black</material>
+        </gazebo>
+        <!-- <gazebo reference="${robot_name}_line_lidar_1">
+            <sensor name="laser_${robot_name}" type="ray">
+                <pose> 0 0 0 0 0 0 </pose>
+                <always_on>true</always_on>
+                <visualize>true</visualize>
+                <update_rate>10</update_rate>
+                <ray>
+                    <scan>
+                        <horizontal>
+                            <samples>360</samples>
+                            <min_angle>-3.14</min_angle>
+                            <max_angle>3.14</max_angle>
+                        </horizontal>
+                    </scan>
+                    <range>
+                        <min>0.3</min>
+                        <max>150</max>
+                    </range>
+                </ray>
+                <plugin name="laser_controller_${robot_name}" filename="libgazebo_ros_ray_sensor.so">
+                    <ros>
+                        <namespace>${robot_name}</namespace>
+                        <argument>~/out:=scan</argument>
+                    </ros>
+                    <output_type>sensor_msgs/LaserScan</output_type>
+                    <frame_name>${robot_name}_line_lidar_1</frame_name>
+                </plugin>
+            </sensor>
+        </gazebo> -->
+        <gazebo reference="${robot_name}_laser_frame_under">
+            <sensor name="laser_${robot_name}" type="ray">
+                <pose> 0 0 0 0 0 0 </pose>
+                <always_on>true</always_on>
+                <visualize>true</visualize>
+                <update_rate>10</update_rate>
+                <ray>
+                    <scan>
+                        <horizontal>
+                            <samples>360</samples>
+                            <min_angle>-1.4</min_angle>
+                            <max_angle>1.4</max_angle>
+                        </horizontal>
+                    </scan>
+                    <range>
+                        <min>0.3</min>
+                        <max>150</max>
+                    </range>
+                </ray>
+                <plugin name="laser_controller_${robot_name}" filename="libgazebo_ros_ray_sensor.so">
+                    <ros>
+                        <namespace>${robot_name}</namespace>
+                        <argument>~/out:=scan</argument>
+                    </ros>
+                    <output_type>sensor_msgs/LaserScan</output_type>
+                    <frame_name>${robot_name}_laser_frame_under</frame_name>
+                </plugin>
+            </sensor>
+        </gazebo>
+        <!-- <gazebo reference="${robot_name}_imu_link">
+            <gravity>true</gravity>
+            <sensor name="imu_sensor" type="imu">
+                <always_on>true</always_on>
+                <update_rate>100</update_rate>
+                <visualize>true</visualize>
+                <topic>imu</topic>
+                <plugin filename="libgazebo_ros_imu_sensor.so" name="imu_plugin">
+                    <topicName>imu</topicName>
+                    <bodyName>${robot_name}_imu_link</bodyName>
+                    <updateRateHZ>100.0</updateRateHZ>
+                    <xyzOffset>0 0 0</xyzOffset>
+                    <rpyOffset>0 0 0</rpyOffset>
+                    <frameName>${robot_name}_imu_link</frameName>
+                    <initialOrientationAsReference>false</initialOrientationAsReference>
+                    <ros>
+                        <namespace>${robot_name}/imu</namespace>
+                        <remapping>~/out:=data</remapping>
+                    </ros>
+                </plugin>
+                <pose>0 0 0 0 0 0</pose>
+            </sensor>
+        </gazebo> -->
+    </xacro:macro>
 </robot>

File: warehouse_bot/urdf/robot_control_gazebo.xacro (robot description, xacro)
@@ -49,9 +49,11 @@
                 <ros>
                     <namespace>${robot_name}</namespace>
+                    <remapping>/tf:=tf</remapping>
+                    <remapping>/tf_static:=tf_static</remapping>
                 </ros>
                 <parameters>$(find warehouse_bot)/robots_config/${robot_name}_controller.yaml</parameters>
                 <robot_param_node>/${robot_name}_robot_state_publisher</robot_param_node>
             </plugin>
-    </gazebo>
+        </gazebo>
     </xacro:macro >
 </robot>

File: warehouse_bot/urdf/robots.urdf.xacro (robot description, xacro)
@@ -231,3 +231,4 @@
     </joint>
   <xacro:robot_gazebo_systems robot_name="$(arg robot_name)"/>
+  <xacro:robot_gazebo_plugins robot_name="$(arg robot_name)"/>
 </robot>
