Commit message: new controller and spawn multi robots

File: livox_laser_simulation_ros2/urdf/mid360.xacro (robot description, xacro)
@@ -66,5 +66,5 @@
 			  </noise>
 			</ray>
-          <visualize>false</visualize>
+          <visualize>true</visualize>
 		  <samples>${samples}</samples>
 		  <downsample>1</downsample>

File: warehouse_bot/urdf/gazebo_control.xacro (robot description, xacro)
@@ -1,8 +1,41 @@
 <?xml version="1.0"?>
-<robot>
+<robot name="warehouse_bot" xmlns:xacro="http://ros.org/wiki/xacro">
+    <!-- Gazebo references -->
+    <gazebo reference="chassis">
+        <mu1 value="0.0" />
+        <mu2 value="0.0" />
+        <kp value="10000000.0" />
+        <kd value="1.0" />
+        <material>Gazebo/Grey</material>
+    </gazebo>
+    <gazebo reference="front_wheel_link">
+        <mu1 value="1.0" />
+        <mu2 value="1.0" />
+        <kp value="10000000.0" />
+        <kd value="1.0" />
+        <fdir1 value="0 0 1" />
+        <material>Gazebo/Black</material>
+    </gazebo>
+    <gazebo reference="lr_wheel_link">
+        <mu1 value="1.0" />
+        <mu2 value="1.0" />
+        <kp value="10000000.0" />
+        <kd value="1.0" />
+        <fdir1 value="1 0 0" />
+        <material>Gazebo/Black</material>
+    </gazebo>
+    <gazebo reference="rr_wheel_link">
+        <mu1 value="1.0" />
+        <mu2 value="1.0" />
+        <kp value="10000000.0" />
+        <kd value="1.0" />
+        <fdir1 value="1 0 0" />
+        <material>Gazebo/Black</material>
+    </gazebo>
     <gazebo reference="line_lidar_1">
         <sensor name="laser1" type="ray">
             <pose> 0 0 0 0 0 0 </pose>
-            <visualize>false</visualize>
+            <always_on>true</always_on>
+            <visualize>true</visualize>
             <update_rate>10</update_rate>
             <ray>
@@ -21,5 +54,5 @@
             <plugin name="laser_controller1" filename="libgazebo_ros_ray_sensor.so">
                 <ros>
-                    <argument>~/out:=scan1</argument>
+                    <argument>~/out:=scan</argument>
                 </ros>
                 <output_type>sensor_msgs/LaserScan</output_type>
@@ -31,5 +64,5 @@
         <sensor name="laser2" type="ray">
             <pose> 0 0 0 0 0 0 </pose>
-            <visualize>false</visualize>
+            <visualize>true</visualize>
             <update_rate>10</update_rate>
             <ray>
@@ -55,3 +88,27 @@
         </sensor>
     </gazebo>
+        <gazebo reference="imu_link">
+        <gravity>true</gravity>
+        <sensor name="imu_sensor" type="imu">
+        <always_on>true</always_on>
+        <update_rate>100</update_rate>
+        <visualize>true</visualize>
+        <topic>imu</topic>
+        <plugin filename="libgazebo_ros_imu_sensor.so" name="imu_plugin">
+            <topicName>imu</topicName>
+            <bodyName>imu_link</bodyName>
+            <updateRateHZ>100.0</updateRateHZ>
+            <!-- <gaussianNoise>0.0</gaussianNoise> -->
+            <xyzOffset>0 0 0</xyzOffset>
+            <rpyOffset>0 0 0</rpyOffset>
+            <frameName>imu_link</frameName>
+            <initialOrientationAsReference>false</initialOrientationAsReference>
+            <ros>
+                <namespace>/imu</namespace>
+                <remapping>~/out:=data</remapping>
+            </ros>
+        </plugin>
+        <pose>0 0 0 0 0 0</pose>
+        </sensor>
+    </gazebo>
 </robot>

File: warehouse_bot/urdf/robot.urdf.xacro (robot description, xacro)
@@ -1,10 +1,12 @@
 <?xml version="1.0"?>
-<robot xmlns:xacro="http://www.ros.org/wiki/xacro"  name="robot">
-    <xacro:include filename="$(find ros2_livox_simulation)/urdf/mid360.xacro" />
+<robot name="robot_1" xmlns:xacro="http://ros.org/wiki/xacro">
+    <!-- <xacro:include filename="$(find ros2_livox_simulation)/urdf/mid360.xacro" />
     <xacro:include filename="$(find warehouse_bot)/urdf/_d435.urdf2.xacro" />
     <xacro:include filename="$(find warehouse_bot)/urdf/_d435.urdf1.xacro" />
-    <xacro:include filename="$(find warehouse_bot)/urdf/_d435.urdf3.xacro" />
-    <xacro:include filename="warehouse_bot.xacro" />
-    <xacro:include filename="ros2_control.xacro" />
-    <xacro:include filename="gazebo_control.xacro" />
+    <xacro:include filename="$(find warehouse_bot)/urdf/_d435.urdf3.xacro" /> -->
+    <xacro:include filename="$(find warehouse_bot)/urdf/materials.xacro" />
+    <xacro:include filename="$(find warehouse_bot)/urdf/macros.xacro" />
+    <xacro:include filename="$(find warehouse_bot)/urdf/ros2_control.xacro" />
+    <xacro:include filename="$(find warehouse_bot)/urdf/warehouse_bot.xacro" />
+    <xacro:include filename="$(find warehouse_bot)/urdf/gazebo_control.xacro" />
 </robot>

File: warehouse_bot/urdf/ros2_control.xacro (robot description, xacro)
@@ -5,12 +5,32 @@
             <plugin>gazebo_ros2_control/GazeboSystem</plugin>
         </hardware>
-        <joint name="steering_joint">
-            <command_interface name="position" />
+        <!-- velocity controller -->
+        <joint name="lr_wheel_joint">
+            <command_interface name="velocity" />
             <state_interface name="position" />
+            <state_interface name="velocity" />
+            <state_interface name="effort" />
         </joint>
-        <joint name="traction_joint">
-                <command_interface name="velocity" />
+        <joint name="rr_wheel_joint">
+            <command_interface name="velocity" />
+            <state_interface name="position" />
             <state_interface name="velocity" />
+            <state_interface name="effort" />
+        </joint>
+        <joint name="front_wheel_joint">
+            <command_interface name="velocity" />
             <state_interface name="position" />
+            <state_interface name="velocity" />
+            <state_interface name="effort" />
+        </joint>
+        <!-- position controller for steering -->
+        <joint name="front_steering_hinge_joint">
+            <command_interface name="position">
+                <param name="min">-0.5</param>
+                <param name="max">0.5</param>
+            </command_interface>
+            <state_interface name="position" />
+            <state_interface name="velocity" />
+            <state_interface name="effort" />
         </joint>
     </ros2_control>

File: warehouse_bot/urdf/warehouse_bot.xacro (robot description, xacro)
@@ -1,4 +1,4 @@
 <?xml version="1.0"?>
-<robot name="warehouse_bot" xmlns:xacro="http://ros.org/wiki/xacro">
+<robot name="robot_1" xmlns:xacro="http://ros.org/wiki/xacro">
     <material name="Black">
       <color rgba="0 0 0 1" />
@@ -13,11 +13,9 @@
       <color rgba="1 1 1 1" />
     </material>
-    <link name="base_link">
-    </link>
     <link name="base_footprint">
     </link>
     <joint name="base_footprint_joint" type="fixed">
-      <parent link="base_link"/>
-      <child link="base_footprint"/>
+      <parent link="base_footprint"/>
+      <child link="chassis"/>
       <origin xyz="0 0 0" rpy="0 0 0"/>
     </joint>
@@ -43,93 +41,41 @@
       </inertial>
     </link>
-    <joint name="chassis_joint" type="fixed">
-      <origin xyz="0 0 0" rpy="0 0 0" />
-      <parent link="base_link" />
-      <child link="chassis" />
-    </joint>
-    <!-- left wheel Link -->
-    <link name="left_wheel">
-      <collision>
-        <geometry>
-          <cylinder length="0.04" radius="0.075" />
-        </geometry>
-      </collision>
-      <visual>
-        <geometry>
-          <cylinder length="0.04" radius="0.075" />
-        </geometry>
-        <material name="Black" />
-      </visual>
-      <inertial>
-        <mass value="50" />
-        <inertia ixx="0.145833" ixy="0.0" ixz="0.0" iyy="0.145833" iyz="0.0" izz="0.125" />
-      </inertial>
-    </link>
-    <joint name="left_wheel_joint" type="continuous">
-      <origin xyz="0 0.2 0" rpy="-1.57 0 0" />
-      <parent link="chassis" />
-      <child link="left_wheel" />
-      <axis xyz="0 0 1" />
-      <dynamics damping="0.2" />
-    </joint>
-    <!-- right wheel Link -->
-    <link name="right_wheel">
-      <collision>
-        <geometry>
-          <cylinder length="0.04" radius="0.075" />
-        </geometry>
-      </collision>
-      <visual>
-        <geometry>
-          <cylinder length="0.04" radius="0.075" />
-        </geometry>
-        <material name="Black" />
-      </visual>
-      <inertial>
-        <mass value="50" />
-        <inertia ixx="0.145833" ixy="0.0" ixz="0.0" iyy="0.145833" iyz="0.0" izz="0.125" />
-      </inertial>
-    </link>
-    <joint name="right_wheel_joint" type="continuous">
-      <origin xyz="0 -0.2 0" rpy="-1.57 0 0" />
-      <parent link="chassis" />
-      <child link="right_wheel" />
-      <axis xyz="0 0 1" />
-      <dynamics damping="0.2" />
-    </joint>
-    <!-- Steering Link -->
-    <link name="steering_link">
-      <visual>
-        <geometry>
-          <box size="0.01 0.01 0.01" />
-        </geometry>
-        <material name="Black" />
-      </visual>
+        <!-- Front Steering Hinge Link -->
+    <link name="front_steering_hinge_link">
       <inertial>
         <origin xyz="0 0 0" rpy="0 0 0" />
-        <mass value="1" />
-        <inertia ixx="0.1" ixy="0.0" ixz="0.0" iyy="0.1" iyz="0.0" izz="0.1" />
+        <mass value="50" />
+        <inertia ixx="4E-06" ixy="0" ixz="0" iyy="4E-06" iyz="0" izz="4E-06" />
       </inertial>
-    </link>
-    <joint name="steering_joint" type="continuous">
+      <visual>
+        <origin xyz="0 0 0" rpy="0 0 0" />
+        <geometry>
+          <box size="0.005 0.005 0.005"/>
+        </geometry>
+      </visual>
+    </link>
+    <joint name="front_steering_hinge_joint" type="revolute">
       <origin xyz="1.1 0 0" rpy="0 0 0" />
       <parent link="chassis" />
-      <child link="steering_link" />
+      <child link="front_steering_hinge_link" />
       <axis xyz="0 0 1" />
+      <limit lower="-0.7853" upper="0.7853" effort="10" velocity="100" />
     </joint>
-    <!-- traction wheel link -->
-    <link name="wheel_front_link">
+    <!-- Front Wheel Link -->
+    <link name="front_wheel_link">
+      <inertial>
+        <origin xyz="0.0 0.0 0.0" rpy="0 0 0"/>
+        <mass value="2"/>
+        <inertia ixx="0.00025" iyy="0.00014" izz="0.00014" ixy="0.0" iyz="0.0" ixz="0.0"/>
+      </inertial>
       <visual>
+        <origin xyz="0 0 0" rpy="0 0 0"/>
         <geometry>
           <cylinder length="0.05" radius="0.075" />
         </geometry>
-        <material name="Black" />
+        <material name="black"/>
       </visual>
-      <inertial>
-        <origin xyz="0 0 0" rpy="0 0 0" />
-        <mass value="100" />
-        <inertia ixx="1" ixy="0" ixz="0" iyy="1" iyz="0" izz="1" />
-      </inertial>
       <collision>
+        <origin xyz="0 0 0" rpy="0 0 0"/>
         <geometry>
           <cylinder length="0.05" radius="0.075" />
@@ -137,10 +83,76 @@
       </collision>
     </link>
-    <joint name="traction_joint" type="continuous">
-      <parent link="steering_link" />
-      <child link="wheel_front_link" />
-      <origin xyz="0 0 0" rpy="-1.57 1.57 0" />
+    <joint name="front_wheel_joint" type="continuous">
+      <origin xyz="0.0 0.0 0.0" rpy="-1.57 1.57 0" />
+      <parent link="front_steering_hinge_link" />
+      <child link="front_wheel_link" />
       <axis xyz="0 0 1" />
+      <limit effort="10" velocity="100" />
     </joint>
+  <!-- Rear Left Wheel Link -->
+  <link name="lr_wheel_link">
+    <inertial>
+      <origin xyz="0.0 0.0 0.0" rpy="0 0 0"/>
+      <mass value="2"/>
+      <inertia ixx="0.00025" iyy="0.00014" izz="0.00014" ixy="0.0" iyz="0.0" ixz="0.0"/>
+    </inertial>
+    <visual>
+        <geometry>
+          <cylinder length="0.04" radius="0.075" />
+        </geometry>
+      <material name="black"/>
+    </visual>
+    <collision>
+      <origin xyz="0 0 0" rpy="0 0 0"/>
+        <geometry>
+          <cylinder length="0.04" radius="0.075" />
+        </geometry>
+    </collision>
+  </link>
+  <joint name="lr_wheel_joint" type="continuous">
+    <origin xyz="0 0.2 0" rpy="-1.57 0 0" />
+    <parent link="chassis" />
+    <child link="lr_wheel_link" />
+    <axis xyz="0 0 1" />
+  </joint>
+  <!-- Rear Right Wheel Link -->
+  <link name="rr_wheel_link">
+    <inertial>
+      <origin xyz="0.0 0.0 0.0" rpy="0 0 0"/>
+      <mass value="0.20069792517970372"/>
+      <inertia ixx="0.00025" iyy="0.00014" izz="0.00014" ixy="0.0" iyz="0.0" ixz="0.0"/>
+    </inertial>
+    <visual>
+      <origin xyz="0 0 0" rpy="0 0 0"/>
+        <geometry>
+          <cylinder length="0.04" radius="0.075" />
+        </geometry>
+      <material name="black"/>
+    </visual>
+    <collision>
+      <origin xyz="0 0 0" rpy="0 0 0"/>
+        <geometry>
+          <cylinder length="0.04" radius="0.075" />
+        </geometry>
+    </collision>
+  </link>
+  <joint name="rr_wheel_joint" type="continuous">
+    <origin xyz="0 -0.2 0" rpy="-1.57 0 0" />
+    <parent link="chassis" />
+    <child link="rr_wheel_link" />
+    <axis xyz="0 0 1" />
+  </joint>
+  <!-- IMU Link -->
+  <link name="imu_link">
+    <inertial>
+      <mass value="0.01"/>
+      <inertia ixx="1.0" ixy="0" ixz="0" iyy="1.0" iyz="0" izz="1.0"/>
+    </inertial>
+  </link>
+  <joint name="imu_joint" type="fixed">
+    <origin xyz="0.2715 0 0.041" rpy="0 0 0"/>
+    <parent link="chassis"/>
+    <child link="imu_link"/>
+  </joint>
   <link name="line_lidar_1">
     <inertial>
@@ -162,23 +174,4 @@
     </collision>
   </link>
-  <!-- <link name="mid-360-asm_1">
-    <inertial>
-      <origin xyz="0 0 0" rpy="0 0 0"/>
-      <mass value="0.01"/>
-      <inertia ixx="0.1" ixy="0.0" ixz="0.0" iyy="0.1" iyz="0.0" izz="0.155" />
-    </inertial>
-    <visual>
-      <origin xyz="1.195 0.0 -1.7" rpy="0 0 3.14"/>
-      <geometry>
-        <mesh filename="file://$(find warehouse_bot)/meshes/mid-360-asm_1.stl" scale="0.001 0.001 0.001"/>
-      </geometry>
-    </visual>
-    <collision>
-      <origin xyz="1.195 0.0 -1.7" rpy="0 0 3.14"/>
-      <geometry>
-        <mesh filename="file://$(find warehouse_bot)/meshes/mid-360-asm_1.stl" scale="0.001 0.001 0.001"/>
-      </geometry>
-    </collision>
-  </link> -->
   <link name="laser_frame_under">
     <inertial>
@@ -221,21 +214,16 @@
   <joint name="fork_joint" type="fixed">
     <origin xyz="0.0 0.0 0.022893" rpy="0 0 0"/>
-    <parent link="base_link"/>
+    <parent link="chassis"/>
     <child link="fork_1"/>
   </joint>
-  <xacro:sensor_d435_1 name="camera1" topics_ns="camera1" parent="base_link" publish_pointcloud="true">
+  <!-- <xacro:sensor_d435_1 name="camera1" topics_ns="camera1" parent="chassis" publish_pointcloud="true">
     <origin xyz="-0.46 0.19 0.05" rpy="0 0 3.14" />
   </xacro:sensor_d435_1>
-  <xacro:sensor_d435_2 name="camera2" topics_ns="camera2" parent="base_link" publish_pointcloud="true">
+  <xacro:sensor_d435_2 name="camera2" topics_ns="camera2" parent="chassis" publish_pointcloud="true">
     <origin xyz="-0.46 -0.19 0.05" rpy="0 0 3.14" />
   </xacro:sensor_d435_2>
-  <xacro:sensor_d435_3 name="camera3" topics_ns="camera3" parent="base_link" publish_pointcloud="true">
+  <xacro:sensor_d435_3 name="camera3" topics_ns="camera3" parent="chassis" publish_pointcloud="true">
     <origin xyz="1.0 0.0 1.77" rpy="0 2.2 3.14" />
-  </xacro:sensor_d435_3>
-  <!-- <joint name="mid360_joint" type="fixed">
-    <origin xyz="1.175 0.0 1.68" rpy="0 0 0"/>
-    <parent link="chassis"/>
-    <child link="mid-360-asm_1"/>
-  </joint>  -->
+  </xacro:sensor_d435_3>   -->
   <joint name="16line_lidar_joint" type="fixed">
     <origin xyz="1.1 0.0 2.24" rpy="0 0 0"/>
@@ -248,6 +236,6 @@
     <child link="laser_frame_under"/>
   </joint>
-  <xacro:mid360 name="livox" parent="base_link" topic="mid360">
+  <!-- <xacro:mid360 name="livox" parent="chassis" topic="mid360">
     <origin xyz="1.175 0.0 1.67" rpy="3.14 0 0"/>
-  </xacro:mid360>
+  </xacro:mid360> -->
 </robot>
