Commit message: fix bug with namespaces for ros2 control

File: multi_robots_rmf_nav2/urdf/gazebo_control.xacro (robot description, xacro)
@@ -1,113 +1,115 @@
 <?xml version="1.0"?>
 <robot name="warehouse_bot" xmlns:xacro="http://ros.org/wiki/xacro">
-    <!-- Gazebo references -->
-    <gazebo reference="chassis">
-        <mu1 value="0.0" />
-        <mu2 value="0.0" />
-        <kp value="10000000.0" />
-        <kd value="1.0" />
-        <material>Gazebo/Grey</material>
-    </gazebo>
-    <gazebo reference="front_wheel_link">
-        <mu1 value="1.0" />
-        <mu2 value="1.0" />
-        <kp value="10000000.0" />
-        <kd value="1.0" />
-        <fdir1 value="0 0 1" />
-        <material>Gazebo/Black</material>
-    </gazebo>
-    <gazebo reference="lr_wheel_link">
-        <mu1 value="1.0" />
-        <mu2 value="1.0" />
-        <kp value="10000000.0" />
-        <kd value="1.0" />
-        <fdir1 value="1 0 0" />
-        <material>Gazebo/Black</material>
-    </gazebo>
-    <gazebo reference="rr_wheel_link">
-        <mu1 value="1.0" />
-        <mu2 value="1.0" />
-        <kp value="10000000.0" />
-        <kd value="1.0" />
-        <fdir1 value="1 0 0" />
-        <material>Gazebo/Black</material>
-    </gazebo>
-    <!-- <gazebo reference="line_lidar_1">
-        <sensor name="laser1" type="ray">
-            <pose> 0 0 0 0 0 0 </pose>
+    <xacro:macro  name="robot_gazebo_sensors" params="robot_name">
+        <!-- Gazebo references -->
+        <gazebo reference="chassis">
+            <mu1 value="0.0" />
+            <mu2 value="0.0" />
+            <kp value="10000000.0" />
+            <kd value="1.0" />
+            <material>Gazebo/Grey</material>
+        </gazebo>
+        <gazebo reference="front_wheel_link">
+            <mu1 value="1.0" />
+            <mu2 value="1.0" />
+            <kp value="10000000.0" />
+            <kd value="1.0" />
+            <fdir1 value="0 0 1" />
+            <material>Gazebo/Black</material>
+        </gazebo>
+        <gazebo reference="lr_wheel_link">
+            <mu1 value="1.0" />
+            <mu2 value="1.0" />
+            <kp value="10000000.0" />
+            <kd value="1.0" />
+            <fdir1 value="1 0 0" />
+            <material>Gazebo/Black</material>
+        </gazebo>
+        <gazebo reference="rr_wheel_link">
+            <mu1 value="1.0" />
+            <mu2 value="1.0" />
+            <kp value="10000000.0" />
+            <kd value="1.0" />
+            <fdir1 value="1 0 0" />
+            <material>Gazebo/Black</material>
+        </gazebo>
+        <!-- <gazebo reference="line_lidar_1">
+            <sensor name="laser1" type="ray">
+                <pose> 0 0 0 0 0 0 </pose>
+                <always_on>true</always_on>
+                <visualize>false</visualize>
+                <update_rate>10</update_rate>
+                <ray>
+                    <scan>
+                        <horizontal>
+                            <samples>360</samples>
+                            <min_angle>-3.14</min_angle>
+                            <max_angle>3.14</max_angle>
+                        </horizontal>
+                    </scan>
+                    <range>
+                        <min>0.3</min>
+                        <max>15.0</max>
+                    </range>
+                </ray>
+                <plugin name="laser_controller1" filename="libgazebo_ros_ray_sensor.so">
+                    <ros>
+                        <remapping>~/out:=scan</remapping>
+                    </ros>
+                    <output_type>sensor_msgs/LaserScan</output_type>
+                    <frame_name>line_lidar_1</frame_name>
+                </plugin>
+            </sensor>
+        </gazebo> -->
+        <gazebo reference="laser_frame_under">
+            <sensor name="${robot_name}_laser2" type="ray">
+                <pose> 0 0 0 0 0 0 </pose>
+                <visualize>true</visualize>
+                <update_rate>10</update_rate>
+                <ray>
+                    <scan>
+                        <horizontal>
+                            <samples>360</samples>
+                            <min_angle>-2.4</min_angle>
+                            <max_angle>2.4</max_angle>
+                        </horizontal>
+                    </scan>
+                    <range>
+                        <min>0.3</min>
+                        <max>15.0</max>
+                    </range>
+                </ray>
+                <plugin name="${robot_name}_laser_controller2" filename="libgazebo_ros_ray_sensor.so">
+                    <ros>
+                        <remapping>~/out:=scan2</remapping>
+                    </ros>
+                    <output_type>sensor_msgs/LaserScan</output_type>
+                    <frame_name>laser_frame_under</frame_name>
+                </plugin>
+            </sensor>
+        </gazebo>
+            <gazebo reference="imu_link">
+            <gravity>true</gravity>
+            <sensor name="${robot_name}_imu_sensor" type="imu">
             <always_on>true</always_on>
-            <visualize>false</visualize>
-            <update_rate>10</update_rate>
-            <ray>
-                <scan>
-                    <horizontal>
-                        <samples>360</samples>
-                        <min_angle>-3.14</min_angle>
-                        <max_angle>3.14</max_angle>
-                    </horizontal>
-                </scan>
-                <range>
-                    <min>0.3</min>
-                    <max>15.0</max>
-                </range>
-            </ray>
-            <plugin name="laser_controller1" filename="libgazebo_ros_ray_sensor.so">
+            <update_rate>100</update_rate>
+            <visualize>true</visualize>
+            <topic>imu</topic>
+            <plugin filename="libgazebo_ros_imu_sensor.so" name="${robot_name}_imu_plugin">
+                <topicName>imu</topicName>
+                <bodyName>imu_link</bodyName>
+                <updateRateHZ>100.0</updateRateHZ>
+                <gaussianNoise>0.0</gaussianNoise>
+                <xyzOffset>0 0 0</xyzOffset>
+                <rpyOffset>0 0 0</rpyOffset>
+                <frameName>imu_link</frameName>
+                <initialOrientationAsReference>false</initialOrientationAsReference>
                 <ros>
-                    <remapping>~/out:=scan</remapping>
+                    <remapping>~/out:=imu</remapping>
                 </ros>
-                <output_type>sensor_msgs/LaserScan</output_type>
-                <frame_name>line_lidar_1</frame_name>
             </plugin>
-        </sensor>
-    </gazebo> -->
-    <gazebo reference="laser_frame_under">
-        <sensor name="laser2" type="ray">
-            <pose> 0 0 0 0 0 0 </pose>
-            <visualize>true</visualize>
-            <update_rate>10</update_rate>
-            <ray>
-                <scan>
-                    <horizontal>
-                        <samples>360</samples>
-                        <min_angle>-2.4</min_angle>
-                        <max_angle>2.4</max_angle>
-                    </horizontal>
-                </scan>
-                <range>
-                    <min>0.3</min>
-                    <max>15.0</max>
-                </range>
-            </ray>
-            <plugin name="laser_controller2" filename="libgazebo_ros_ray_sensor.so">
-                <ros>
-                    <remapping>~/out:=scan2</remapping>
-                </ros>
-                <output_type>sensor_msgs/LaserScan</output_type>
-                <frame_name>laser_frame_under</frame_name>
-            </plugin>
-        </sensor>
-    </gazebo>
-           <gazebo reference="imu_link">
-        <gravity>true</gravity>
-        <sensor name="imu_sensor" type="imu">
-        <always_on>true</always_on>
-        <update_rate>100</update_rate>
-        <visualize>true</visualize>
-        <topic>imu</topic>
-        <plugin filename="libgazebo_ros_imu_sensor.so" name="imu_plugin">
-            <topicName>imu</topicName>
-            <bodyName>imu_link</bodyName>
-            <updateRateHZ>100.0</updateRateHZ>
-            <gaussianNoise>0.0</gaussianNoise>
-            <xyzOffset>0 0 0</xyzOffset>
-            <rpyOffset>0 0 0</rpyOffset>
-            <frameName>imu_link</frameName>
-            <initialOrientationAsReference>false</initialOrientationAsReference>
-            <ros>
-                <remapping>~/out:=imu</remapping>
-            </ros>
-        </plugin>
-        <pose>0 0 0 0 0 0</pose>
-        </sensor>
-    </gazebo>
+            <pose>0 0 0 0 0 0</pose>
+            </sensor>
+        </gazebo>
+    </xacro:macro >
 </robot>

File: multi_robots_rmf_nav2/urdf/robot.urdf.xacro (robot description, xacro)
@@ -1,4 +1,5 @@
 <?xml version="1.0"?>
 <robot name="robot_1" xmlns:xacro="http://ros.org/wiki/xacro">
+    <xacro:arg name="robot_name" default="robot1"/>
     <!-- <xacro:include filename="$(find ros2_livox_simulation)/urdf/mid360.xacro" />
     <xacro:include filename="$(find multi_robots_rmf_nav2)/urdf/_d435.urdf2.xacro" />
@@ -6,8 +7,11 @@
     <xacro:include filename="$(find multi_robots_rmf_nav2)/urdf/_d435.urdf3.xacro" />
     <xacro:include filename="$(find robosense_description)/urdf/RS-16.urdf.xacro"/> -->
-    <xacro:include filename="$(find multi_robots_rmf_nav2)/urdf/materials.xacro" />
-    <xacro:include filename="$(find multi_robots_rmf_nav2)/urdf/macros.xacro" />
-    <xacro:include filename="$(find multi_robots_rmf_nav2)/urdf/ros2_control.xacro" />
-    <xacro:include filename="$(find multi_robots_rmf_nav2)/urdf/warehouse_bot.xacro" />
-    <xacro:include filename="$(find multi_robots_rmf_nav2)/urdf/gazebo_control.xacro" />
+    <!-- Определение аргумента для namespace с дефолтным значением -->
+    <xacro:include filename="$(find multi_robots_rmf_nav2)/urdf/materials.xacro"/>
+    <xacro:include filename="$(find multi_robots_rmf_nav2)/urdf/macros.xacro"/>
+    <xacro:include filename="$(find multi_robots_rmf_nav2)/urdf/warehouse_bot.xacro"/>
+    <xacro:include filename="$(find multi_robots_rmf_nav2)/urdf/gazebo_control.xacro"/>
+    <xacro:include filename="$(find multi_robots_rmf_nav2)/urdf/ros2_control.xacro"/>
+    <xacro:robot_gazebo_systems robot_name="$(arg robot_name)"/>
+    <xacro:robot_gazebo_sensors robot_name="$(arg robot_name)"/>
 </robot>

File: multi_robots_rmf_nav2/urdf/ros2_control.xacro (robot description, xacro)
@@ -1,42 +1,46 @@
-<?xml version="1.0"?>
-<robot name="warehouse_bot" xmlns:xacro="http://ros.org/wiki/xacro">
-    <ros2_control name="GazeboSystem" type="system">
-        <hardware>
-            <plugin>gazebo_ros2_control/GazeboSystem</plugin>
-        </hardware>
-        <!-- velocity controller -->
-        <joint name="lr_wheel_joint">
-            <command_interface name="velocity" />
-            <state_interface name="position" />
-            <state_interface name="velocity" />
-            <state_interface name="effort" />
-        </joint>
-        <joint name="rr_wheel_joint">
-            <command_interface name="velocity" />
-            <state_interface name="position" />
-            <state_interface name="velocity" />
-            <state_interface name="effort" />
-        </joint>
-        <joint name="front_wheel_joint">
-            <command_interface name="velocity" />
-            <state_interface name="position" />
-            <state_interface name="velocity" />
-            <state_interface name="effort" />
-        </joint>
-        <!-- position controller for steering -->
-        <joint name="front_steering_hinge_joint">
-            <command_interface name="position">
-                <param name="min">-0.5</param>
-                <param name="max">0.5</param>
-            </command_interface>
-            <state_interface name="position" />
-            <state_interface name="velocity" />
-            <state_interface name="effort" />
-        </joint>
-    </ros2_control>
-    <gazebo>
-        <plugin name="robot_gazebo_ros2_control" filename="libgazebo_ros2_control.so">
-            <parameters>$(find multi_robots_rmf_nav2)/config/tricycle_drive_controller.yaml</parameters>
-        </plugin>
-    </gazebo>
+<robot xmlns:xacro="http://www.ros.org/wiki/xacro">
+    <xacro:macro  name="robot_gazebo_systems" params="robot_name">
+        <ros2_control name="${robot_name}_GazeboSystem" type="system">
+            <hardware>
+                <plugin>gazebo_ros2_control/GazeboSystem</plugin>
+            </hardware>
+            <!-- velocity controller -->
+            <joint name="lr_wheel_joint">
+                <command_interface name="velocity" />
+                <state_interface name="position" />
+                <state_interface name="velocity" />
+                <state_interface name="effort" />
+            </joint>
+            <joint name="rr_wheel_joint">
+                <command_interface name="velocity" />
+                <state_interface name="position" />
+                <state_interface name="velocity" />
+                <state_interface name="effort" />
+            </joint>
+            <joint name="front_wheel_joint">
+                <command_interface name="velocity" />
+                <state_interface name="position" />
+                <state_interface name="velocity" />
+                <state_interface name="effort" />
+            </joint>
+            <!-- position controller for steering -->
+            <joint name="front_steering_hinge_joint">
+                <command_interface name="position">
+                    <param name="min">-0.5</param>
+                    <param name="max">0.5</param>
+                </command_interface>
+                <state_interface name="position" />
+                <state_interface name="velocity" />
+                <state_interface name="effort" />
+            </joint>
+        </ros2_control>
+        <gazebo>
+            <plugin filename="libgazebo_ros2_control.so" name="${robot_name}_gazebo_ros2_control">
+                <ros>
+                    <namespace>/${robot_name}</namespace>
+                </ros>
+                <parameters>$(find multi_robots_rmf_nav2)/config/tricycle_drive_controller.yaml</parameters>
+            </plugin>
+        </gazebo>
+    </xacro:macro >
 </robot>

Commit message: update 10 robots rmf nav2

File: multi_robots_rmf_nav2/urdf/gazebo_control.xacro (robot description, xacro)
@@ -63,51 +63,38 @@
         </gazebo> -->
         <gazebo reference="laser_frame_under">
-            <sensor name="${robot_name}_laser2" type="ray">
+            <!--<material>Gazebo/Black</material>-->
+            <sensor name="laser" type="gpu_lidar">
                 <pose> 0 0 0 0 0 0 </pose>
-                <visualize>true</visualize>
+                <visualize>false</visualize>
                 <update_rate>10</update_rate>
-                <ray>
+                <lidar>
                     <scan>
                         <horizontal>
                             <samples>360</samples>
-                            <min_angle>-2.4</min_angle>
-                            <max_angle>2.4</max_angle>
+                            <min_angle>-3.14</min_angle>
+                            <max_angle>3.14</max_angle>
                         </horizontal>
                     </scan>
                     <range>
-                        <min>0.3</min>
-                        <max>15.0</max>
+                        <min>0.12</min>
+                        <max>12</max>
                     </range>
-                </ray>
-                <plugin name="${robot_name}_laser_controller2" filename="libgazebo_ros_ray_sensor.so">
-                    <ros>
-                        <remapping>~/out:=scan2</remapping>
-                    </ros>
-                    <output_type>sensor_msgs/LaserScan</output_type>
-                    <frame_name>laser_frame_under</frame_name>
-                </plugin>
+                </lidar>
+                <topic>/${robot_name}/scan2</topic>
+                <gz_frame_id>laser_frame_under</gz_frame_id>
             </sensor>
         </gazebo>
-            <gazebo reference="imu_link">
-            <gravity>true</gravity>
-            <sensor name="${robot_name}_imu_sensor" type="imu">
-            <always_on>true</always_on>
-            <update_rate>100</update_rate>
-            <visualize>true</visualize>
-            <topic>imu</topic>
-            <plugin filename="libgazebo_ros_imu_sensor.so" name="${robot_name}_imu_plugin">
-                <topicName>imu</topicName>
-                <bodyName>imu_link</bodyName>
-                <updateRateHZ>100.0</updateRateHZ>
-                <gaussianNoise>0.0</gaussianNoise>
-                <xyzOffset>0 0 0</xyzOffset>
-                <rpyOffset>0 0 0</rpyOffset>
-                <frameName>imu_link</frameName>
-                <initialOrientationAsReference>false</initialOrientationAsReference>
-                <ros>
-                    <remapping>~/out:=imu</remapping>
-                </ros>
-            </plugin>
-            <pose>0 0 0 0 0 0</pose>
+        <gazebo reference="imu_link">
+            <!--<material>Gazebo/Black</material>-->
+            <gravity>false</gravity>
+            <sensor name="imu_sensor" type="imu">
+                <always_on>true</always_on>
+                <update_rate>100</update_rate>
+                <visualize>false</visualize>
+                <topic>/${robot_name}/imu</topic>
+                    <plugin filename="libgz-sim-imu-system.so" name="gz::sim::systems::Imu">
+                </plugin>
+                <pose>0 0 0 0 0 0</pose>
+                <gz_frame_id>imu_link</gz_frame_id> <!-- Добавьте этот тег для указания кадра -->
             </sensor>
         </gazebo>

File: multi_robots_rmf_nav2/urdf/ros2_control.xacro (robot description, xacro)
@@ -1,7 +1,7 @@
 <robot xmlns:xacro="http://www.ros.org/wiki/xacro">
     <xacro:macro  name="robot_gazebo_systems" params="robot_name">
-        <ros2_control name="${robot_name}_GazeboSystem" type="system">
+        <ros2_control name="${robot_name}_IgnitionSystem" type="system">
             <hardware>
-                <plugin>gazebo_ros2_control/GazeboSystem</plugin>
+                <plugin>ign_ros2_control/IgnitionSystem</plugin>
             </hardware>
             <!-- velocity controller -->
@@ -36,5 +36,5 @@
         </ros2_control>
         <gazebo>
-            <plugin filename="libgazebo_ros2_control.so" name="${robot_name}_gazebo_ros2_control">
+            <plugin filename="ign_ros2_control-system" name="ign_ros2_control::IgnitionROS2ControlPlugin">
                 <ros>
                     <namespace>/${robot_name}</namespace>

File: multi_robots_rmf_nav2/urdf/warehouse_bot.xacro (robot description, xacro)
@@ -15,10 +15,18 @@
       <color rgba="1 1 1 1" />
     </material>
+    <link name="base_link">
+    </link>
+    <!-- BASE_FOOTPRINT LINK -->
+    <joint name="base_footprint_joint" type="fixed">
+        <parent link="base_link"/>
+        <child link="base_footprint"/>
+        <origin xyz="0 0 0" rpy="0 0 0"/>
+    </joint>
     <link name="base_footprint">
     </link>
-    <joint name="base_footprint_joint" type="fixed">
-      <parent link="base_footprint"/>
-      <child link="chassis"/>
-      <origin xyz="0 0 0" rpy="0 0 0"/>
+    <joint name="chassis_joint" type="fixed">
+        <parent link="base_link"/>
+        <child link="chassis"/>
+        <origin xyz="0 0 0"/>
     </joint>
     <!-- Chassis -->
